File: stm32_calc/stm32_calc.kicad_sch (KiCad schematic)
At the start: 75 parts, among them IC1 TM1638, J2 Conn_01x03, J4 C5307759, J4 Conn_02x03_Odd_Even, Q1 p channel mosfet sot 23, SW1 Reset, SW1 batter_switch, SW2 SS-1290, U1 STM32F072CBT6, U1 XC6206P332MR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

Commit message: updated pcb
Parts:
- added H1, H2, H3, H4, H5, H6: MountingHole_Pad, MountingHole:MountingHole_2.2mm_M2_DIN965_Pad, symbol Mechanical:MountingHole_Pad
Connections:
- no-connect marks 27 -> 33
Changed lines of the file:
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@@
   (no_connect (at 210.82 135.89))
   (no_connect (at 288.29 91.44))
+  (no_connect (at 350.52 262.89))
+  (no_connect (at 299.72 262.89))
   (no_connect (at 163.83 55.88))
   (no_connect (at 210.82 123.19))
@@
   (no_connect (at 176.53 55.88))
   (no_connect (at 189.23 55.88))
+  (no_connect (at 374.65 262.89))
   (no_connect (at 252.73 101.6))
   (no_connect (at 144.78 55.88))
@@
   (no_connect (at 123.19 83.82))
   (no_connect (at 252.73 91.44))
+  (no_connect (at 274.32 262.89))
+  (no_connect (at 247.65 262.89))
   (no_connect (at 170.18 143.51))
   (no_connect (at 182.88 55.88))
   (no_connect (at 170.18 55.88))
   (no_connect (at 123.19 96.52))
+  (no_connect (at 325.12 262.89))
   (wire (pts (xy 278.13 139.7) (xy 278.13 143.51))
     (stroke (width 0) (type default))
@@
     )
   )
+  (symbol (lib_id "Mechanical:MountingHole_Pad") (at 247.65 260.35 0) (unit 1)
+    (in_bom yes) (on_board yes) (dnp no) (fields_autoplaced)
+    (property "Reference" "H1" (at 250.19 257.81 0)
+      (effects (font (size 1.27 1.27)) (justify left))
+    )
+    (property "Value" "MountingHole_Pad" (at 250.19 260.35 0)
+      (effects (font (size 1.27 1.27)) (justify left))
+    )
+    (property "Footprint" "MountingHole:MountingHole_2.2mm_M2_DIN965_Pad" (at 247.65 260.35 0)
+      (effects (font (size 1.27 1.27)) hide)
+    )
+    (property "Datasheet" "~" (at 247.65 260.35 0)
+      (effects (font (size 1.27 1.27)) hide)
+    )
+    (pin "1")
+    (instances
+      (project "stm32_calc"
+        (path "/fc977c70-bd16-408a-afd0-76aeebefb268"
+          (reference "H1") (unit 1)
+        )
+      )
+    )
+  )
   (symbol (lib_id "Device:R") (at 452.12 166.37 0) (unit 1)
     (in_bom yes) (on_board yes) (dnp no) (fields_autoplaced)
@@
     )
   )
+  (symbol (lib_id "Mechanical:MountingHole_Pad") (at 374.65 260.35 0) (unit 1)
+    (in_bom yes) (on_board yes) (dnp no) (fields_autoplaced)
+    (property "Reference" "H6" (at 377.19 257.81 0)
+      (effects (font (size 1.27 1.27)) (justify left))
+    )
+    (property "Value" "MountingHole_Pad" (at 377.19 260.35 0)
+      (effects (font (size 1.27 1.27)) (justify left))
+    )
+    (property "Footprint" "MountingHole:MountingHole_2.2mm_M2_DIN965_Pad" (at 374.65 260.35 0)
+      (effects (font (size 1.27 1.27)) hide)
+    )
+    (property "Datasheet" "~" (at 374.65 260.35 0)
+      (effects (font (size 1.27 1.27)) hide)
+    )
+    (pin "1")
+    (instances
+      (project "stm32_calc"
+        (path "/fc977c70-bd16-408a-afd0-76aeebefb268"
+          (reference "H6") (unit 1)
+        )
+      )
+    )
+  )
   (symbol (lib_id "Device:C") (at 328.93 195.58 0) (unit 1)
     (in_bom yes) (on_board yes) (dnp no)
@@
     )
   )
+  (symbol (lib_id "Mechanical:MountingHole_Pad") (at 350.52 260.35 0) (unit 1)
+    (in_bom yes) (on_board yes) (dnp no) (fields_autoplaced)
+    (property "Reference" "H5" (at 353.06 257.81 0)
+      (effects (font (size 1.27 1.27)) (justify left))
+    )
+    (property "Value" "MountingHole_Pad" (at 353.06 260.35 0)
+      (effects (font (size 1.27 1.27)) (justify left))
+    )
+    (property "Footprint" "MountingHole:MountingHole_2.2mm_M2_DIN965_Pad" (at 350.52 260.35 0)
+      (effects (font (size 1.27 1.27)) hide)
+    )
+    (property "Datasheet" "~" (at 350.52 260.35 0)
+      (effects (font (size 1.27 1.27)) hide)
+    )
+    (pin "1")
+    (instances
+      (project "stm32_calc"
+        (path "/fc977c70-bd16-408a-afd0-76aeebefb268"
+          (reference "H5") (unit 1)
+        )
+      )
+    )
+  )
   (symbol (lib_id "Device:R") (at 438.15 185.42 90) (unit 1)
     (in_bom yes) (on_board yes) (dnp no)
@@
     )
   )
+  (symbol (lib_id "Mechanical:MountingHole_Pad") (at 325.12 260.35 0) (unit 1)
+    (in_bom yes) (on_board yes) (dnp no) (fields_autoplaced)
+    (property "Reference" "H4" (at 327.66 257.81 0)
+      (effects (font (size 1.27 1.27)) (justify left))
+    )
+    (property "Value" "MountingHole_Pad" (at 327.66 260.35 0)
+      (effects (font (size 1.27 1.27)) (justify left))
+    )
+    (property "Footprint" "MountingHole:MountingHole_2.2mm_M2_DIN965_Pad" (at 325.12 260.35 0)
+      (effects (font (size 1.27 1.27)) hide)
+    )
+    (property "Datasheet" "~" (at 325.12 260.35 0)
+      (effects (font (size 1.27 1.27)) hide)
+    )
+    (pin "1")
+    (instances
+      (project "stm32_calc"
+        (path "/fc977c70-bd16-408a-afd0-76aeebefb268"
+          (reference "H4") (unit 1)
+        )
+      )
+    )
+  )
   (symbol (lib_id "Switch:SW_SPST") (at 476.25 90.17 0) (unit 1)
     (in_bom yes) (on_board yes) (dnp no) (fields_autoplaced)
@@
     )
   )
+  (symbol (lib_id "Mechanical:MountingHole_Pad") (at 299.72 260.35 0) (unit 1)
+    (in_bom yes) (on_board yes) (dnp no) (fields_autoplaced)
+    (property "Reference" "H3" (at 302.26 257.81 0)
+      (effects (font (size 1.27 1.27)) (justify left))
+    )
+    (property "Value" "MountingHole_Pad" (at 302.26 260.35 0)
+      (effects (font (size 1.27 1.27)) (justify left))
+    )
+    (property "Footprint" "MountingHole:MountingHole_2.2mm_M2_DIN965_Pad" (at 299.72 260.35 0)
+      (effects (font (size 1.27 1.27)) hide)
+    )
+    (property "Datasheet" "~" (at 299.72 260.35 0)
+      (effects (font (size 1.27 1.27)) hide)
+    )
+    (pin "1")
+    (instances
+      (project "stm32_calc"
+        (path "/fc977c70-bd16-408a-afd0-76aeebefb268"
+          (reference "H3") (unit 1)
+        )
+      )
+    )
+  )
   (symbol (lib_id "power:GND") (at 273.05 241.3 0) (unit 1)
     (in_bom yes) (on_board yes) (dnp no) (fields_autoplaced)
@@
         )
       )
+    )
+  )
+  (symbol (lib_id "Mechanical:MountingHole_Pad") (at 274.32 260.35 0) (unit 1)
+    (in_bom yes) (on_board yes) (dnp no) (fields_autoplaced)
+    (property "Reference" "H2" (at 276.86 257.81 0)
+      (effects (font (size 1.27 1.27)) (justify left))
+    )
+    (property "Value" "MountingHole_Pad" (at 276.86 260.35 0)
+      (effects (font (size 1.27 1.27)) (justify left))
+    )
+    (property "Footprint" "MountingHole:MountingHole_2.2mm_M2_DIN965_Pad" (at 274.32 260.35 0)
+      (effects (font (size 1.27 1.27)) hide)
+    )
+    (property "Datasheet" "~" (at 274.32 260.35 0)
+      (effects (font (size 1.27 1.27)) hide)
+    )
+    (pin "1")
+    (instances
+      (project "stm32_calc"
+        (path "/fc977c70-bd16-408a-afd0-76aeebefb268"
+          (reference "H2") (unit 1)
+        )
+      )

Commit message: added switch and bottom plate
Parts:
- J4: footprint Connector_USB:USB_C_Receptacle_G-Switch_GT-USB-7010ASV -> Connector_USB:USB_C_Receptacle_HRO_TYPE-C-31-M-12
Changed lines of the file:
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@@
       (effects (font (size 1.27 1.27)))
     )
-    (property "Footprint" "Connector_USB:USB_C_Receptacle_G-Switch_GT-USB-7010ASV" (at 422.91 193.04 0)
+    (property "Footprint" "Connector_USB:USB_C_Receptacle_HRO_TYPE-C-31-M-12" (at 422.91 193.04 0)
       (effects (font (size 1.27 1.27)) hide)
     )

Commit message: updated pcb
Parts:
- added C9: 100n, Capacitor_SMD:C_0402_1005Metric, symbol Device:C_Small
- D21: value 1n4001 -> 1n4148
Connections:
- net DBUS+ is gone; now on net D+: J4.A6 (D+), J4.B6 (D+), U2.4 (I/O2)
- net DBUS- is gone; now on net D-: J4.A7 (D-), J4.B7 (D-), U2.6 (I/O1)
- net +3V3: now also C9.1
- net GND: now also C9.2
Changed lines of the file:
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@@
   (junction (at 433.07 97.79) (diameter 0) (color 0 0 0 0)
   )
+  (junction (at 278.13 140.97) (diameter 0) (color 0 0 0 0)
+  )
   (junction (at 118.745 109.22) (diameter 0) (color 0 0 0 0)
   )
@@
   (no_connect (at 123.19 96.52))
   (no_connect (at 325.12 262.89))
-  (wire (pts (xy 278.13 139.7) (xy 278.13 143.51))
+  (wire (pts (xy 278.13 139.7) (xy 278.13 140.97))
     (stroke (width 0) (type default))
   )
@@
     (stroke (width 0) (type default))
   )
+  (wire (pts (xy 278.13 140.97) (xy 278.13 143.51))
+    (stroke (width 0) (type default))
+  )
   (wire (pts (xy 201.93 148.59) (xy 201.93 155.575))
     (stroke (width 0) (type solid))
@@
     (stroke (width 0) (type solid))
   )
+  (wire (pts (xy 281.94 143.51) (xy 281.94 140.97))
+    (stroke (width 0) (type default))
+  )
   (wire (pts (xy 328.93 190.5) (xy 335.28 190.5))
     (stroke (width 0) (type default))
@@
     (stroke (width 0) (type default))
   )
+  (wire (pts (xy 271.78 140.97) (xy 271.78 142.24))
+    (stroke (width 0) (type default))
+  )
   (wire (pts (xy 222.885 71.755) (xy 222.885 72.39))
     (stroke (width 0) (type solid))
@@
     (stroke (width 0) (type default))
   )
-  (wire (pts (xy 285.75 140.97) (xy 285.75 143.51))
-    (stroke (width 0) (type default))
-  )
   (wire (pts (xy 500.38 38.1) (xy 500.38 49.53))
     (stroke (width 0) (type default))
@@
     (stroke (width 0) (type solid))
   )
-  (wire (pts (xy 278.13 143.51) (xy 285.75 143.51))
-    (stroke (width 0) (type default))
-  )
   (wire (pts (xy 452.12 57.15) (xy 471.17 57.15))
     (stroke (width 0) (type default))
@@
     (stroke (width 0) (type default))
   )
+  (wire (pts (xy 278.13 143.51) (xy 281.94 143.51))
+    (stroke (width 0) (type default))
+  )
   (wire (pts (xy 443.23 69.85) (xy 443.23 90.17))
     (stroke (width 0) (type default))
@@
     (stroke (width 0) (type default))
   )
+  (wire (pts (xy 273.05 140.97) (xy 271.78 140.97))
+    (stroke (width 0) (type default))
+  )
   (rectangle (start 400.05 13.97) (end 516.89 146.05)
     (stroke (width 0) (type default))
@@
     )
   )
+  (global_label "D+" (shape input) (at 502.92 198.12 0) (fields_autoplaced)
+    (effects (font (size 1.27 1.27)) (justify left))
+    (property "Intersheetrefs" "${INTERSHEET_REFS}" (at 508.7476 198.12 0)
+      (effects (font (size 1.27 1.27)) (justify left) hide)
+    )
+  )
   (global_label "col0" (shape input) (at 163.83 143.51 270) (fields_autoplaced)
     (effects (font (size 1.27 1.27)) (justify right))
@@
     )
   )
+  (global_label "D+" (shape input) (at 445.77 198.12 0) (fields_autoplaced)
+    (effects (font (size 1.27 1.27)) (justify left))
+    (property "Intersheetrefs" "${INTERSHEET_REFS}" (at 451.5976 198.12 0)
+      (effects (font (size 1.27 1.27)) (justify left) hide)
+    )
+  )
   (global_label "GR1" (shape input) (at 312.42 48.26 180) (fields_autoplaced)
     (effects (font (size 1.27 1.27)) (justify right))
@@
     )
   )
-  (global_label "DBUS-" (shape input) (at 482.6 198.12 180) (fields_autoplaced)
+  (global_label "col1" (shape input) (at 157.48 143.51 270) (fields_autoplaced)
     (effects (font (size 1.27 1.27)) (justify right))
-    (property "Intersheetrefs" "${INTERSHEET_REFS}" (at 472.9624 198.12 0)
+    (property "Intersheetrefs" "${INTERSHEET_REFS}" (at 157.48 150.6075 90)
       (effects (font (size 1.27 1.27)) (justify right) hide)
     )
   )
-  (global_label "col1" (shape input) (at 157.48 143.51 270) (fields_autoplaced)
+  (global_label "D-" (shape input) (at 482.6 198.12 180) (fields_autoplaced)
     (effects (font (size 1.27 1.27)) (justify right))
-    (property "Intersheetrefs" "${INTERSHEET_REFS}" (at 157.48 150.6075 90)
+    (property "Intersheetrefs" "${INTERSHEET_REFS}" (at 476.7724 198.12 0)
       (effects (font (size 1.27 1.27)) (justify right) hide)
     )
@@
     )
   )
-  (global_label "DBUS+" (shape input) (at 445.77 198.12 0) (fields_autoplaced)
-    (effects (font (size 1.27 1.27)) (justify left))
-    (property "Intersheetrefs" "${INTERSHEET_REFS}" (at 455.4076 198.12 0)
-      (effects (font (size 1.27 1.27)) (justify left) hide)
-    )
-  )
   (global_label "D+" (shape input) (at 210.82 85.09 0) (fields_autoplaced)
     (effects (font (size 1.27 1.27)) (justify left))
@@
     )
   )
-  (global_label "DBUS-" (shape input) (at 445.77 193.04 0) (fields_autoplaced)
+  (global_label "D-" (shape input) (at 445.77 193.04 0) (fields_autoplaced)
     (effects (font (size 1.27 1.27)) (justify left))
-    (property "Intersheetrefs" "${INTERSHEET_REFS}" (at 455.4076 193.04 0)
+    (property "Intersheetrefs" "${INTERSHEET_REFS}" (at 451.5976 193.04 0)
       (effects (font (size 1.27 1.27)) (justify left) hide)
     )
@@
     )
   )
-  (global_label "DBUS+" (shape input) (at 502.92 198.12 0) (fields_autoplaced)
-    (effects (font (size 1.27 1.27)) (justify left))
-    (property "Intersheetrefs" "${INTERSHEET_REFS}" (at 512.5576 198.12 0)
-      (effects (font (size 1.27 1.27)) (justify left) hide)
-    )
-  )
   (global_label "CLK" (shape input) (at 270.51 26.67 90) (fields_autoplaced)
     (effects (font (size 1.27 1.27)) (justify left))
@@
       (effects (font (size 1.27 1.27)))
     )
-    (property "Value" "1n4001" (at 304.8 186.69 0)
+    (property "Value" "1n4148" (at 304.8 186.69 0)
       (effects (font (size 1.27 1.27)))
     )
@@
     )
   )
+  (symbol (lib_id "power:GND") (at 271.78 142.24 0) (unit 1)
+    (in_bom yes) (on_board yes) (dnp no)
+    (property "Reference" "#PWR010" (at 271.78 148.59 0)
+      (effects (font (size 1.27 1.27)) hide)
+    )
+    (property "Value" "GND" (at 271.78 139.7 0)
+      (effects (font (size 1.27 1.27)))
+    )
+    (property "Footprint" "" (at 271.78 142.24 0)
+      (effects (font (size 1.27 1.27)) hide)
+    )
+    (property "Datasheet" "" (at 271.78 142.24 0)
+      (effects (font (size 1.27 1.27)) hide)
+    )
+    (pin "1")
+    (instances
+      (project "mech_calc"
+        (path "/000044fd-33a1-4b17-8153-101e1c8b9dc1"
+          (reference "#PWR010") (unit 1)
+        )
+      )
+      (project "rp2040_calc"
+        (path "/c1c20588-ed59-444c-9775-23c5bb4a512e"
+          (reference "#PWR028") (unit 1)
+        )
+      )
+      (project "stm32_calc"
+        (path "/fc977c70-bd16-408a-afd0-76aeebefb268"
+          (reference "#PWR035") (unit 1)
+        )
+      )
+    )
+  )
   (symbol (lib_id "Switch:SW_SPST") (at 457.2 49.53 0) (unit 1)
     (in_bom yes) (on_board yes) (dnp no) (fields_autoplaced)
@@
     )
   )
-  (symbol (lib_id "power:+3V3") (at 285.75 140.97 0) (unit 1)
+  (symbol (lib_id "power:+3V3") (at 281.94 140.97 0) (unit 1)
     (in_bom yes) (on_board yes) (dnp no)
-    (property "Reference" "#PWR09" (at 285.75 144.78 0)
+    (property "Reference" "#PWR09" (at 281.94 144.78 0)
       (effects (font (size 1.27 1.27)) hide)
     )
-    (property "Value" "+3V3" (at 286.131 136.5758 0)
+    (property "Value" "+3V3" (at 282.321 136.5758 0)
       (effects (font (size 1.27 1.27)))
     )
-    (property "Footprint" "" (at 285.75 140.97 0)
+    (property "Footprint" "" (at 281.94 140.97 0)
       (effects (font (size 1.27 1.27)) hide)
     )
-    (property "Datasheet" "" (at 285.75 140.97 0)
+    (property "Datasheet" "" (at 281.94 140.97 0)
       (effects (font (size 1.27 1.27)) hide)
     )
@@
         )
       )
+    )
+  )
+  (symbol (lib_id "Device:C_Small") (at 275.59 140.97 270) (unit 1)
+    (in_bom yes) (on_board yes) (dnp no)
+    (property "Reference" "C9" (at 275.59 144.78 90)
+      (effects (font (size 0.7874 0.7874)))
+    )
+    (property "Value" "100n" (at 275.59 143.51 90)
+      (effects (font (size 0.7874 0.7874)))
+    )
+    (property "Footprint" "Capacitor_SMD:C_0402_1005Metric" (at 275.59 140.97 0)
+      (effects (font (size 1.27 1.27)) hide)
+    )
+    (property "Datasheet" "~" (at 275.59 140.97 0)
+      (effects (font (size 1.27 1.27)) hide)
+    )
+    (property "Package" "C0402" (at 275.59 140.97 0)
+      (effects (font (size 1.27 1.27)) hide)
+    )
+    (pin "1")
+    (pin "2")
+    (instances
+      (project "fluxon"
+        (path "/25ab855a-c74b-4020-b9dd-0dd3df5942a0"
+          (reference "C9") (unit 1)
+        )
+      )
+      (project "stm32_calc"
+        (path "/fc977c70-bd16-408a-afd0-76aeebefb268"
+          (reference "C11") (unit 1)
+        )
+      )

Commit message: fixed resistor footprints
Parts:
- C4, C5, C6: footprint Capacitor_SMD:C_0805_2012Metric -> Capacitor_SMD:C_0402_1005Metric
- R1, R10, R11, R12, R13, R2, R3, R4, R7: footprint Capacitor_SMD:C_0402_1005Metric -> Resistor_SMD:R_0402_1005Metric
Changed lines of the file:
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@@
       (effects (font (size 1.27 1.27)) (justify left))
     )
-    (property "Footprint" "Capacitor_SMD:C_0402_1005Metric" (at 450.342 166.37 90)
+    (property "Footprint" "Resistor_SMD:R_0402_1005Metric" (at 450.342 166.37 90)
       (effects (font (size 1.27 1.27)) hide)
     )
@@
       (effects (font (size 1.27 1.27)))
     )
-    (property "Footprint" "Capacitor_SMD:C_0402_1005Metric" (at 266.7 231.648 90)
+    (property "Footprint" "Resistor_SMD:R_0402_1005Metric" (at 266.7 231.648 90)
       (effects (font (size 1.27 1.27)) hide)
     )
@@
       (effects (font (size 1.27 1.27)))
     )
-    (property "Footprint" "Capacitor_SMD:C_0402_1005Metric" (at 438.15 187.198 90)
+    (property "Footprint" "Resistor_SMD:R_0402_1005Metric" (at 438.15 187.198 90)
       (effects (font (size 1.27 1.27)) hide)
     )
@@
       (effects (font (size 1.27 1.27)) (justify left))
     )
-    (property "Footprint" "Capacitor_SMD:C_0402_1005Metric" (at 450.342 173.99 90)
+    (property "Footprint" "Resistor_SMD:R_0402_1005Metric" (at 450.342 173.99 90)
       (effects (font (size 1.27 1.27)) hide)
     )
@@
       (effects (font (size 1.27 1.27)))
     )
-    (property "Footprint" "Capacitor_SMD:C_0805_2012Metric" (at 259.08 37.1348 0)
+    (property "Footprint" "Capacitor_SMD:C_0402_1005Metric" (at 259.08 37.1348 0)
       (effects (font (size 1.27 1.27)) hide)
     )
@@
       (effects (font (size 1.27 1.27)) (justify left))
     )
-    (property "Footprint" "Capacitor_SMD:C_0402_1005Metric" (at 290.322 200.66 90)
+    (property "Footprint" "Resistor_SMD:R_0402_1005Metric" (at 290.322 200.66 90)
       (effects (font (size 1.27 1.27)) hide)
     )
@@
       (effects (font (size 1.27 1.27)))
     )
-    (property "Footprint" "Capacitor_SMD:C_0402_1005Metric" (at 290.83 30.988 90)
+    (property "Footprint" "Resistor_SMD:R_0402_1005Metric" (at 290.83 30.988 90)
       (effects (font (size 1.27 1.27)) hide)
     )
@@
       (effects (font (size 1.27 1.27)))
     )
-    (property "Footprint" "Capacitor_SMD:C_0805_2012Metric" (at 259.08 28.2448 0)
+    (property "Footprint" "Capacitor_SMD:C_0402_1005Metric" (at 259.08 28.2448 0)
       (effects (font (size 1.27 1.27)) hide)
     )
@@
       (effects (font (size 1.27 1.27)))
     )
-    (property "Footprint" "Capacitor_SMD:C_0402_1005Metric" (at 438.15 184.658 90)
+    (property "Footprint" "Resistor_SMD:R_0402_1005Metric" (at 438.15 184.658 90)
       (effects (font (size 1.27 1.27)) hide)
     )
@@
       (effects (font (size 1.27 1.27)))
     )
-    (property "Footprint" "Capacitor_SMD:C_0402_1005Metric" (at 290.83 39.878 90)
+    (property "Footprint" "Resistor_SMD:R_0402_1005Metric" (at 290.83 39.878 90)
       (effects (font (size 1.27 1.27)) hide)
     )
@@
       (effects (font (size 1.27 1.27)))
     )
-    (property "Footprint" "Capacitor_SMD:C_0805_2012Metric" (at 259.08 46.0248 0)
+    (property "Footprint" "Capacitor_SMD:C_0402_1005Metric" (at 259.08 46.0248 0)
       (effects (font (size 1.27 1.27)) hide)
     )
@@
       (effects (font (size 1.27 1.27)))
     )
-    (property "Footprint" "Capacitor_SMD:C_0402_1005Metric" (at 318.77 232.918 90)
+    (property "Footprint" "Resistor_SMD:R_0402_1005Metric" (at 318.77 232.918 90)
       (effects (font (size 1.27 1.27)) hide)
     )
@@
       (effects (font (size 1.27 1.27)))
     )
-    (property "Footprint" "Capacitor_SMD:C_0402_1005Metric" (at 290.83 48.768 90)
+    (property "Footprint" "Resistor_SMD:R_0402_1005Metric" (at 290.83 48.768 90)
       (effects (font (size 1.27 1.27)) hide)
     )

Commit message: updated pcb
Connections:
- net usb_check_mcu: now also U1.41 (SPI1_MOSI/I2S1_SD/TIM3_CH2/PB5); no longer U1.22 (PB11/TIM2_CH4/I2C2_SDA)
Changed lines of the file:
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@@
   (junction (at 247.65 38.1) (diameter 0) (color 0 0 0 0)
   )
+  (no_connect (at 189.23 143.51))
   (no_connect (at 288.29 93.98))
   (no_connect (at 252.73 96.52))
@@
   (no_connect (at 123.19 77.47))
   (no_connect (at 210.82 129.54))
-  (no_connect (at 176.53 55.88))
   (no_connect (at 189.23 55.88))
   (no_connect (at 374.65 262.89))
@@
     )
   )
-  (global_label "usb_check_mcu" (shape input) (at 189.23 143.51 270) (fields_autoplaced)
-    (effects (font (size 1.27 1.27)) (justify right))
-    (property "Intersheetrefs" "${INTERSHEET_REFS}" (at 189.23 161.1303 90)
-      (effects (font (size 1.27 1.27)) (justify right) hide)
-    )
-  )
+  (global_label "usb_check_mcu" (shape input) (at 176.53 55.88 90) (fields_autoplaced)
+    (effects (font (size 1.27 1.27)) (justify left))
+    (property "Intersheetrefs" "${INTERSHEET_REFS}" (at 176.53 38.2597 90)
+      (effects (font (size 1.27 1.27)) (justify left) hide)
+    )
+  )
