File: stm32_calc/stm32_calc.kicad_sch (KiCad schematic)
At the start: 82 parts, among them IC1 TM1638, J2 Conn_01x03, J4 C5307759, J4 Conn_02x03_Odd_Even, Q1 p channel mosfet sot 23, SW1 Reset, SW1 batter_switch, SW2 SS-1290, U1 STM32F072CBT6, U1 XC6206P332MR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

Commit message: added graphics, fixed some tracing
Parts:
- D1, D10, D11, D12, D13, D14, D16, D17, D19, D2, D20, D21, D3, D4, D5, D6, D7, D8, D9: footprint Diode_SMD:Nexperia_CFP3_SOD-123W -> Diode_SMD:D_SOD-123
Connections:
- net col0: now also U1.16 (PA6/ADC_IN6/TIM3_CH1/TIM16_CH1); no longer U1.18 (PB0/TIM3_CH3/ADC_IN8)
- net col1: now also U1.15 (PA5/ADC_IN5/DAC_OUT2); no longer U1.17 (PA7/TIM3_CH2/TIM14_CH1/ADC_IN7)
- net col2: now also U1.14 (PA4/TIM14_CH1/ADC_IN4); no longer U1.16 (PA6/ADC_IN6/TIM3_CH1/TIM16_CH1)
- net col3: now also U1.13 (PA3/TIM15_CH2/ADC_IN3); no longer U1.15 (PA5/ADC_IN5/DAC_OUT2)
- net row0: now also U1.17 (PA7/TIM3_CH2/TIM14_CH1/ADC_IN7); no longer U1.14 (PA4/TIM14_CH1/ADC_IN4)
- net row1: now also U1.18 (PB0/TIM3_CH3/ADC_IN8); no longer U1.13 (PA3/TIM15_CH2/ADC_IN3)
Changed lines of the file:
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@@
     )
   )
-  (global_label "col0" (shape input) (at 163.83 143.51 270) (fields_autoplaced)
+  (global_label "col0" (shape input) (at 151.13 143.51 270) (fields_autoplaced)
     (effects (font (size 1.27 1.27)) (justify right))
-    (property "Intersheetrefs" "${INTERSHEET_REFS}" (at 163.83 150.6075 90)
+    (property "Intersheetrefs" "${INTERSHEET_REFS}" (at 151.13 150.6075 90)
       (effects (font (size 1.27 1.27)) (justify right) hide)
     )
@@
     )
   )
-  (global_label "col1" (shape input) (at 157.48 143.51 270) (fields_autoplaced)
+  (global_label "col1" (shape input) (at 144.78 143.51 270) (fields_autoplaced)
     (effects (font (size 1.27 1.27)) (justify right))
-    (property "Intersheetrefs" "${INTERSHEET_REFS}" (at 157.48 150.6075 90)
+    (property "Intersheetrefs" "${INTERSHEET_REFS}" (at 144.78 150.6075 90)
       (effects (font (size 1.27 1.27)) (justify right) hide)
     )
@@
     )
   )
-  (global_label "row0" (shape input) (at 138.43 143.51 270) (fields_autoplaced)
+  (global_label "row0" (shape input) (at 157.48 143.51 270) (fields_autoplaced)
     (effects (font (size 1.27 1.27)) (justify right))
-    (property "Intersheetrefs" "${INTERSHEET_REFS}" (at 138.43 150.9704 90)
+    (property "Intersheetrefs" "${INTERSHEET_REFS}" (at 157.48 150.9704 90)
       (effects (font (size 1.27 1.27)) (justify right) hide)
     )
@@
     )
   )
-  (global_label "row1" (shape input) (at 132.08 143.51 270) (fields_autoplaced)
+  (global_label "row1" (shape input) (at 163.83 143.51 270) (fields_autoplaced)
     (effects (font (size 1.27 1.27)) (justify right))
-    (property "Intersheetrefs" "${INTERSHEET_REFS}" (at 132.08 150.9704 90)
+    (property "Intersheetrefs" "${INTERSHEET_REFS}" (at 163.83 150.9704 90)
       (effects (font (size 1.27 1.27)) (justify right) hide)
     )
@@
     )
   )
-  (global_label "col3" (shape input) (at 144.78 143.51 270) (fields_autoplaced)
+  (global_label "col3" (shape input) (at 132.08 143.51 270) (fields_autoplaced)
     (effects (font (size 1.27 1.27)) (justify right))
-    (property "Intersheetrefs" "${INTERSHEET_REFS}" (at 144.78 150.6075 90)
+    (property "Intersheetrefs" "${INTERSHEET_REFS}" (at 132.08 150.6075 90)
       (effects (font (size 1.27 1.27)) (justify right) hide)
     )
@@
     )
   )
-  (global_label "col2" (shape input) (at 151.13 143.51 270) (fields_autoplaced)
+  (global_label "col2" (shape input) (at 138.43 143.51 270) (fields_autoplaced)
     (effects (font (size 1.27 1.27)) (justify right))
-    (property "Intersheetrefs" "${INTERSHEET_REFS}" (at 151.13 150.6075 90)
+    (property "Intersheetrefs" "${INTERSHEET_REFS}" (at 138.43 150.6075 90)
       (effects (font (size 1.27 1.27)) (justify right) hide)
     )
@@
       (effects (font (size 1.27 1.27)))
     )
-    (property "Footprint" "Diode_SMD:Nexperia_CFP3_SOD-123W" (at 304.8 190.5 0)
+    (property "Footprint" "Diode_SMD:D_SOD-123" (at 304.8 190.5 0)
       (effects (font (size 1.27 1.27)) hide)
     )
@@
       (effects (font (size 1.27 1.27)) (justify right))
     )
-    (property "Footprint" "Diode_SMD:Nexperia_CFP3_SOD-123W" (at 433.07 53.34 0)
+    (property "Footprint" "Diode_SMD:D_SOD-123" (at 433.07 53.34 0)
       (effects (font (size 1.27 1.27)) hide)
     )
@@
       (effects (font (size 1.27 1.27)) (justify right))
     )
-    (property "Footprint" "Diode_SMD:Nexperia_CFP3_SOD-123W" (at 433.07 73.66 0)
+    (property "Footprint" "Diode_SMD:D_SOD-123" (at 433.07 73.66 0)
       (effects (font (size 1.27 1.27)) hide)
     )
@@
       (effects (font (size 1.27 1.27)))
     )
-    (property "Footprint" "Diode_SMD:Nexperia_CFP3_SOD-123W" (at 284.48 182.88 0)
+    (property "Footprint" "Diode_SMD:D_SOD-123" (at 284.48 182.88 0)
       (effects (font (size 1.27 1.27)) hide)
     )
@@
       (effects (font (size 1.27 1.27)) (justify right))
     )
-    (property "Footprint" "Diode_SMD:Nexperia_CFP3_SOD-123W" (at 490.22 114.3 0)
+    (property "Footprint" "Diode_SMD:D_SOD-123" (at 490.22 114.3 0)
       (effects (font (size 1.27 1.27)) hide)
     )
@@
       (effects (font (size 1.27 1.27)) (justify right))
     )
-    (property "Footprint" "Diode_SMD:Nexperia_CFP3_SOD-123W" (at 471.17 134.62 0)
+    (property "Footprint" "Diode_SMD:D_SOD-123" (at 471.17 134.62 0)
       (effects (font (size 1.27 1.27)) hide)
     )
@@
       (effects (font (size 1.27 1.27)) (justify right))
     )
-    (property "Footprint" "Diode_SMD:Nexperia_CFP3_SOD-123W" (at 471.17 114.3 0)
+    (property "Footprint" "Diode_SMD:D_SOD-123" (at 471.17 114.3 0)
       (effects (font (size 1.27 1.27)) hide)
     )
@@
       (effects (font (size 1.27 1.27)) (justify right))
     )
-    (property "Footprint" "Diode_SMD:Nexperia_CFP3_SOD-123W" (at 452.12 73.66 0)
+    (property "Footprint" "Diode_SMD:D_SOD-123" (at 452.12 73.66 0)
       (effects (font (size 1.27 1.27)) hide)
     )
@@
       (effects (font (size 1.27 1.27)) (justify right))
     )
-    (property "Footprint" "Diode_SMD:Nexperia_CFP3_SOD-123W" (at 452.12 93.98 0)
+    (property "Footprint" "Diode_SMD:D_SOD-123" (at 452.12 93.98 0)
       (effects (font (size 1.27 1.27)) hide)
     )
@@
       (effects (font (size 1.27 1.27)) (justify right))
     )
-    (property "Footprint" "Diode_SMD:Nexperia_CFP3_SOD-123W" (at 433.07 134.62 0)
+    (property "Footprint" "Diode_SMD:D_SOD-123" (at 433.07 134.62 0)
       (effects (font (size 1.27 1.27)) hide)
     )
@@
       (effects (font (size 1.27 1.27)) (justify right))
     )
-    (property "Footprint" "Diode_SMD:Nexperia_CFP3_SOD-123W" (at 452.12 114.3 0)
+    (property "Footprint" "Diode_SMD:D_SOD-123" (at 452.12 114.3 0)
       (effects (font (size 1.27 1.27)) hide)
     )
@@
       (effects (font (size 1.27 1.27)) (justify right))
     )
-    (property "Footprint" "Diode_SMD:Nexperia_CFP3_SOD-123W" (at 433.07 93.98 0)
+    (property "Footprint" "Diode_SMD:D_SOD-123" (at 433.07 93.98 0)
       (effects (font (size 1.27 1.27)) hide)
     )
@@
       (effects (font (size 1.27 1.27)) (justify right))
     )
-    (property "Footprint" "Diode_SMD:Nexperia_CFP3_SOD-123W" (at 471.17 73.66 0)
+    (property "Footprint" "Diode_SMD:D_SOD-123" (at 471.17 73.66 0)
       (effects (font (size 1.27 1.27)) hide)
     )
@@
       (effects (font (size 1.27 1.27)) (justify right))
     )
-    (property "Footprint" "Diode_SMD:Nexperia_CFP3_SOD-123W" (at 471.17 93.98 0)
+    (property "Footprint" "Diode_SMD:D_SOD-123" (at 471.17 93.98 0)
       (effects (font (size 1.27 1.27)) hide)
     )
@@
       (effects (font (size 1.27 1.27)) (justify right))
     )
-    (property "Footprint" "Diode_SMD:Nexperia_CFP3_SOD-123W" (at 490.22 53.34 0)
+    (property "Footprint" "Diode_SMD:D_SOD-123" (at 490.22 53.34 0)
       (effects (font (size 1.27 1.27)) hide)
     )
@@
       (effects (font (size 1.27 1.27)) (justify right))
     )
-    (property "Footprint" "Diode_SMD:Nexperia_CFP3_SOD-123W" (at 452.12 53.34 0)
+    (property "Footprint" "Diode_SMD:D_SOD-123" (at 452.12 53.34 0)
       (effects (font (size 1.27 1.27)) hide)
     )
@@
       (effects (font (size 1.27 1.27)) (justify right))
     )
-    (property "Footprint" "Diode_SMD:Nexperia_CFP3_SOD-123W" (at 471.17 53.34 0)
+    (property "Footprint" "Diode_SMD:D_SOD-123" (at 471.17 53.34 0)
       (effects (font (size 1.27 1.27)) hide)
     )
@@
       (effects (font (size 1.27 1.27)) (justify right))
     )
-    (property "Footprint" "Diode_SMD:Nexperia_CFP3_SOD-123W" (at 433.07 114.3 0)
+    (property "Footprint" "Diode_SMD:D_SOD-123" (at 433.07 114.3 0)
       (effects (font (size 1.27 1.27)) hide)
     )
@@
       (effects (font (size 1.27 1.27)) (justify right))
     )
-    (property "Footprint" "Diode_SMD:Nexperia_CFP3_SOD-123W" (at 490.22 73.66 0)
+    (property "Footprint" "Diode_SMD:D_SOD-123" (at 490.22 73.66 0)
       (effects (font (size 1.27 1.27)) hide)
     )

Commit message: updated pcb
Connections:
- net D+: no longer J4.A6 (D+), J4.B6 (D+), U2.3 (I/O2)
- net D-: no longer J4.A7 (D-), J4.B7 (D-), U2.1 (I/O1)
- new net usbD+: J4.A6 (D+), J4.B6 (D+), U2.3 (I/O2)
- new net usbD-: J4.A7 (D-), J4.B7 (D-), U2.1 (I/O1)
Changed lines of the file:
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@@
-    )
-  )
-  (global_label "D+" (shape input) (at 502.92 203.2 0) (fields_autoplaced)
-    (effects (font (size 1.27 1.27)) (justify left))
-    (property "Intersheetrefs" "${INTERSHEET_REFS}" (at 508.7476 203.2 0)
-      (effects (font (size 1.27 1.27)) (justify left) hide)
     )
   )
@@
     )
   )
-  (global_label "D+" (shape input) (at 445.77 198.12 0) (fields_autoplaced)
-    (effects (font (size 1.27 1.27)) (justify left))
-    (property "Intersheetrefs" "${INTERSHEET_REFS}" (at 451.5976 198.12 0)
+  (global_label "usbD+" (shape input) (at 445.77 198.12 0) (fields_autoplaced)
+    (effects (font (size 1.27 1.27)) (justify left))
+    (property "Intersheetrefs" "${INTERSHEET_REFS}" (at 454.9237 198.12 0)
       (effects (font (size 1.27 1.27)) (justify left) hide)
     )
@@
     )
   )
-  (global_label "D-" (shape input) (at 482.6 203.2 180) (fields_autoplaced)
-    (effects (font (size 1.27 1.27)) (justify right))
-    (property "Intersheetrefs" "${INTERSHEET_REFS}" (at 476.7724 203.2 0)
-      (effects (font (size 1.27 1.27)) (justify right) hide)
-    )
-  )
   (global_label "BOOT0" (shape input) (at 157.48 55.88 90) (fields_autoplaced)
     (effects (font (size 1.27 1.27)) (justify left))
@@
     )
   )
-  (global_label "D-" (shape input) (at 445.77 193.04 0) (fields_autoplaced)
-    (effects (font (size 1.27 1.27)) (justify left))
-    (property "Intersheetrefs" "${INTERSHEET_REFS}" (at 451.5976 193.04 0)
+  (global_label "usbD-" (shape input) (at 445.77 193.04 0) (fields_autoplaced)
+    (effects (font (size 1.27 1.27)) (justify left))
+    (property "Intersheetrefs" "${INTERSHEET_REFS}" (at 454.9237 193.04 0)
       (effects (font (size 1.27 1.27)) (justify left) hide)
     )
@@
     )
   )
+  (global_label "usbD+" (shape input) (at 502.92 203.2 0) (fields_autoplaced)
+    (effects (font (size 1.27 1.27)) (justify left))
+    (property "Intersheetrefs" "${INTERSHEET_REFS}" (at 512.0737 203.2 0)
+      (effects (font (size 1.27 1.27)) (justify left) hide)
+    )
+  )
   (global_label "CLK" (shape input) (at 270.51 26.67 90) (fields_autoplaced)
     (effects (font (size 1.27 1.27)) (justify left))
@@
     )
   )
+  (global_label "usbD-" (shape input) (at 482.6 203.2 180) (fields_autoplaced)
+    (effects (font (size 1.27 1.27)) (justify right))
+    (property "Intersheetrefs" "${INTERSHEET_REFS}" (at 473.4463 203.2 0)
+      (effects (font (size 1.27 1.27)) (justify right) hide)
+    )
+  )
