File: stm32_calc/stm32_calc.kicad_pcb (KiCad board)
At the start: 2 copper layers, 76.2 x 132.2 mm, 85 parts, among them IC1 TM1638, J2 Conn_01x03, J3 C5307759, J4 Conn_02x03_Odd_Even, Q1 p channel mosfet sot 23, SW1 batter_switch, SW2 SS-1290, SW3 Reset, U1 STM32F072CBT6, U2 USBLC6-2SC6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

Commit message: updated pcb
Parts:
- removed the G*** at (81.9, 122.2)
- moved J2 4.38 mm to (117.5, 72.3), turned to 180 degrees
- moved R8 0.62 mm to (88.1, 67.7), turned to -90 degrees
- moved R10 0.42 mm to (87.1, 67.7)
- moved R13 0.42 mm to (84.2, 67.7)
Connections:
- J3 pad A6: D+ -> usbD+
- J3 pad A7: D- -> usbD-
- J3 pad B6: D+ -> usbD+
- J3 pad B7: D- -> usbD-
- U2 pad 1: D- -> usbD-
- U2 pad 3: D+ -> usbD+
Routing:
- net D-: track 24.0 -> 13.6 mm
- net vbus: track 54.2 -> 44.9 mm, vias 5 -> 2
- net D+: track 22.3 -> 13.2 mm
- net Net-(J2-Pin_3): track 8.29 -> 16.6 mm
- net usbD-: track 0.00 -> 8.22 mm
- net usbD+: track 0.00 -> 6.81 mm
- net GND: track 58.4 -> 56.2 mm
- net Net-(D1-A): track 11.8 -> 11.3 mm

Commit message: updated pcb
Parts:
- added G***: LOGO, georgs_lib:logo_w65, B.Cu at (85.6, 87.1)
- U1: footprint georgs_lib:STM32L072CBT6 -> Package_QFP:LQFP-48_7x7mm_P0.5mm
- moved D14 14.1 mm to (101.9, 149.3)
- moved D18 12.0 mm to (105.0, 138.6)
- moved H5 4.13 mm to (85.7, 182.4)
- moved H6 3.66 mm to (116.2, 152.4)
- moved H7 3.66 mm to (55.3, 152.4)
- moved R1 0.73 mm to (109.5, 88.2), turned to 180 degrees
- moved R2 0.65 mm to (91.8, 72.8)
Routing:
- net GR7: track 88.1 -> 80.2 mm
- net Net-(D18-A): track 11.0 -> 16.2 mm
- net SEG2: track 17.5 -> 13.1 mm
- net Net-(D14-A): track 5.08 -> 9.45 mm
- net +3V3: track 14.8 -> 11.8 mm
- net GND: track 56.2 -> 53.5 mm, vias 17 -> 19
- net col2: track 106.7 -> 104.2 mm
- net Net-(J2-Pin_3): track 16.6 -> 18.7 mm
- net col1: track 80.1 -> 78.2 mm
- net col0: track 114.8 -> 113.1 mm
- net Net-(D1-A): track 11.3 -> 12.8 mm
- net col3: track 116.3 -> 115.4 mm
- net NRST: track 38.0 -> 37.2 mm
- net GR8: track 74.6 -> 73.9 mm
- net row4: track 166.9 -> 167.5 mm
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Other:
- board text added: "JLCJLCJLCJLC"

Commit message: updated pcb
Routing:
- net Net-(D18-A): track 16.2 -> 5.13 mm
Changed lines of the file:
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@@
     (effects (font (size 1 1) (thickness 0.15)) (justify left bottom mirror))
+  )
+  (dimension (type aligned) (layer "F.Fab")
+    (pts (xy 47.625 60.25) (xy 123.825 60.25))
+    (height -33.05)
+    (gr_text "76.2000 mm" (at 85.725 26.05) (layer "F.Fab")
+      (effects (font (size 1 1) (thickness 0.15)))
+    )
+    (format (prefix "") (suffix "") (units 3) (units_format 1) (precision 4))
+    (style (thickness 0.1) (arrow_length 1.27) (text_position_mode 0) (extension_height 0.58642) (extension_offset 0.5) keep_text_aligned)
   )
   (segment (start 115.625 82.25) (end 117.305 83.93) (width 0.5) (layer "F.Cu") (net 1))
@@
   (segment (start 106.925 109.8) (end 106.98 109.855) (width 0.2) (layer "B.Cu") (net 30))
   (segment (start 106.98 109.855) (end 111.76 109.855) (width 0.2) (layer "B.Cu") (net 30))
-  (segment (start 111.375 135.25) (end 111.76 135.635) (width 0.2) (layer "B.Cu") (net 31))
   (segment (start 106.795 138.43) (end 111.76 138.43) (width 0.2) (layer "B.Cu") (net 31))
   (segment (start 106.675 138.55) (end 106.795 138.43) (width 0.2) (layer "B.Cu") (net 31))
-  (segment (start 111.76 135.635) (end 111.76 138.43) (width 0.2) (layer "B.Cu") (net 31))
-  (segment (start 111.375 127.55) (end 111.375 135.25) (width 0.2) (layer "B.Cu") (net 31))
   (segment (start 111.125 165.65) (end 111.125 175.895) (width 0.2) (layer "B.Cu") (net 32))
   (segment (start 111.125 175.895) (end 111.76 176.53) (width 0.2) (layer "B.Cu") (net 32))
