File: back_plate/back_plate.kicad_pcb (KiCad board)
At the start: 2 copper layers, 76.2 x 132.2 mm, 7 parts

Commit message: updated pcb
Parts:
- added G***: LOGO, georgs_lib:math_signs, F.Cu at (121.8, 102.4)
Routing:
- added copper zone on B.Cu, net (none)

Commit message: updated pcb
Parts:
- removed the G*** at (121.8, 102.4)
- added G***: LOGO, georgs_lib:math_scatter, F.Cu at (107.5, 80.5)
- moved ? 4.13 mm to (119.1, 160.8)
- moved ? 3.66 mm to (88.7, 130.8)
- moved ? 3.66 mm to (149.5, 130.8)
