File: calc_plate/calc_plate.kicad_pcb (KiCad board)
At the start: 2 copper layers, 76.2 x 95.2 mm, 0 parts

Commit message: updated pcb
Parts:
- added G***: LOGO, libraries:logo_small, B.Cu at (85.4, 88.4)
Routing:
- added copper zone on B.Cu, net (none)
- added copper zone on F.Cu, net (none)
Other:
- outline, holes or cut-outs redrawn
- board text added: "JLCJLCJLCJLC"

Commit message: updated pcb
Other:
- board text removed: "JLCJLCJLCJLC"
Changed lines of the file:
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@@
   (gr_line (start 82.415 57.525) (end 82.415 70.525)
     (stroke (width 0.2) (type solid)) (layer "Edge.Cuts"))
-  (gr_text "JLCJLCJLCJLC" (at 97.14 75.5) (layer "B.SilkS")
-    (effects (font (size 0.5 0.5) (thickness 0.125)) (justify left bottom mirror))
-  )
   (zone (net 0) (net_name "") (layer "F.Cu") (hatch edge 0.5)
     (connect_pads (clearance 0.5))
